File: board/board.kicad_sch (KiCad schematic)
At the start: 1 part

Commit message: initial
Parts:
- added J1: 022_battery_cells, on_edge:on_edge_2x05_device, symbol put_on_edge:022_battery_cells
- added J2: 022_battery_cells, on_edge:on_edge_2x05_host, symbol put_on_edge:022_battery_cells
Connections:
- net GND: now also J1.1 (GND), J2.1 (GND)
- new net balancer/C0: J1.2 (C1-), J2.2 (C1-)
- new net balancer/C1: J1.3 (C1+C2-), J2.3 (C1+C2-)
- new net balancer/C2: J1.4 (C2+C3-), J2.4 (C2+C3-)
- new net balancer/C3: J1.5 (C3+4-), J2.5 (C3+4-)
- new net balancer/C4: J1.6 (C4+), J2.6 (C4+)
Other:
- sheet implementation renamed balancer
- sheet balancer: file implementation.kicad_sch -> balancer.kicad_sch
- sheet balancer ports: added C0, C1, C2, C3, C4; removed none
- note removed: "Input connectors go here"
- note removed: "Output connectors go here"
